Commit message: URDF for KapiBara

File: src/workspace/src/kapibara/description/robot_core.xacro (robot description, xacro)
@@ -18,69 +18,226 @@
         <parent link="base_link" />
         <child link="chassis" />
-        <origin xyz="-0.1 0 0" />
+        <origin xyz="0 0 0" />
     </joint>
     <link name="chassis">
         <visual>
-            <origin xyz="0.15 0 0.075" />
-            <geometry>
-                <box size="0.3 0.3 0.15" />
+            <origin xyz="0 0 0" />
+            <geometry>
+                <mesh filename="package://kapibara/meshes/Bottom.stl" scale="0.001 0.001 0.001" />
+            </geometry>
+            <material name="black" />
+        </visual>
+        <collision>
+            <origin xyz="0 0 0" />
+            <geometry>
+                <box size="0.150 0.083 0.033" />
+            </geometry>
+        </collision>
+        <xacro:inertial_box mass="0.65" x="0.15" y="0.083" z="0.033" >
+            <origin xyz="0 0 0" rpy="0 0 0" />
+        </xacro:inertial_box>
+    </link>
+    <!-- Base -->
+    <joint name="base_joint" type="fixed">
+        <parent link="chassis" />
+        <child link="base" />
+        <origin xyz="0.027 0 0.05" />
+    </joint>
+    <link name="base">
+        <visual>
+            <origin xyz="0 0 0.05" />
+            <geometry>
+                <mesh filename="package://kapibara/meshes/Top.stl" scale="0.001 0.001 0.001" />
             </geometry>
             <material name="orange" />
         </visual>
         <collision>
-            <origin xyz="0.15 0 0.075" />
-            <geometry>
-                <box size="0.3 0.3 0.15" />
-            </geometry>
-        </collision>
-        <xacro:inertial_box mass="0.5" x="0.3" y="0.3" z="0.15" >
-            <origin xyz="0.15 0 0.075" rpy="0 0 0" />
+            <origin xyz="0 0 0.05" />
+            <geometry>
+                <box size="0.279 0.134 0.161" />
+            </geometry>
+        </collision>
+        <xacro:inertial_box mass="1.15" x="0.279" y="0.134" z="0.161" >
+            <origin xyz="0 0 0.05" rpy="0 0 0" />
         </xacro:inertial_box>
     </link>
     <!-- LEFT WHEEL LINK -->
-    <joint name="left_wheel_joint" type="continuous">
-        <parent link="base_link"/>
-        <child link="left_wheel"/>
-        <origin xyz="0 0.175 0" rpy="-${pi/2} 0 0" />
-        <axis xyz="0 0 1" />
-    </joint>
-    <link name="left_wheel">
-        <visual>
-            <geometry>
-                <cylinder radius="0.05" length="0.04" />
-            </geometry>
-            <material name="black"/>
-        </visual>
-        <collision>
-            <geometry>
-                <cylinder radius="0.05" length="0.04" />
-            </geometry>
-        </collision>
-        <xacro:inertial_cylinder mass="0.1" length="0.04" radius="0.05">
-            <origin xyz="0 0 0" rpy="0 0 0" />
+    <joint name="wheel_left1_joint" type="continuous">
+        <parent link="chassis" />
+        <child link="left_wheel1" />
+        <axis xyz="0 0 1"/>
+        <origin rpy="${-pi/2} 0 0" xyz="0.065 0.066 0.0165"/>
+    </joint>
+    <link name="left_wheel1">
+        <visual>
+            <origin xyz="0 0 0" />
+            <geometry>
+                <cylinder radius="0.024" length="0.044" />
+            </geometry>
+            <material name="white" />
+        </visual>
+        <collision>
+            <origin xyz="0 0 0" />
+            <geometry>
+                <cylinder radius="0.024" length="0.044" />
+            </geometry>
+        </collision>
+        <xacro:inertial_cylinder mass="0.1" radius="0.024" length="0.044">
+            <origin xyz="0 0 0" rpy="0 0 1" />
+        </xacro:inertial_cylinder>
+    </link>
+    <joint name="wheel_left2_joint" type="continuous">
+        <parent link="chassis" />
+        <child link="left_wheel2" />
+        <axis xyz="0 0 1"/>
+        <origin rpy="${-pi/2} 0 0" xyz="0.005 0.066 0.0165"/>
+    </joint>
+    <link name="left_wheel2">
+        <visual>
+            <origin xyz="0 0 0" />
+            <geometry>
+                <cylinder radius="0.024" length="0.044" />
+            </geometry>
+            <material name="white" />
+        </visual>
+        <collision>
+            <origin xyz="0 0 0" />
+            <geometry>
+                <cylinder radius="0.024" length="0.044" />
+            </geometry>
+        </collision>
+        <xacro:inertial_cylinder mass="0.1" radius="0.024" length="0.044">
+            <origin xyz="0 0 0" rpy="0 0 1" />
+        </xacro:inertial_cylinder>
+    </link>
+    <joint name="wheel_left3_joint" type="continuous">
+        <parent link="chassis" />
+        <child link="left_wheel3" />
+        <axis xyz="0 0 1"/>
+        <origin rpy="${-pi/2} 0 0" xyz="-0.055 0.066 0.0165"/>
+    </joint>
+    <link name="left_wheel3">
+        <visual>
+            <origin xyz="0 0 0" />
+            <geometry>
+                <cylinder radius="0.024" length="0.044" />
+            </geometry>
+            <material name="white" />
+        </visual>
+        <collision>
+            <origin xyz="0 0 0" />
+            <geometry>
+                <cylinder radius="0.024" length="0.044" />
+            </geometry>
+        </collision>
+        <xacro:inertial_cylinder mass="0.1" radius="0.024" length="0.044">
+            <origin xyz="0 0 0" rpy="0 0 1" />
         </xacro:inertial_cylinder>
     </link>
     <!-- RIGHT WHEEL LINK -->
-    <joint name="right_wheel_joint" type="continuous">
-        <parent link="base_link"/>
-        <child link="right_wheel"/>
-        <origin xyz="0 -0.175 0" rpy="-${pi/2} 0 0" />
-        <axis xyz="0 0 -1" />
-    </joint>
-    <link name="right_wheel">
-        <visual>
-            <geometry>
-                <cylinder radius="0.05" length="0.04" />
-            </geometry>
-            <material name="black"/>
-        </visual>
-        <collision>
-            <geometry>
-                <cylinder radius="0.05" length="0.04" />
-            </geometry>
-        </collision>
-        <xacro:inertial_cylinder mass="0.1" length="0.04" radius="0.05">
-            <origin xyz="0 0 0" rpy="0 0 0" />
-        </xacro:inertial_cylinder>
+    <joint name="wheel_right1_joint" type="continuous">
+        <parent link="chassis" />
+        <child link="right_wheel1" />
+        <axis xyz="0 0 1"/>
+        <origin rpy="${-pi/2} 0 0" xyz="0.065 -0.066 0.0165"/>
+    </joint>
+    <link name="right_wheel1">
+        <visual>
+            <origin xyz="0 0 0" />
+            <geometry>
+                <cylinder radius="0.024" length="0.044" />
+            </geometry>
+            <material name="white" />
+        </visual>
+        <collision>
+            <origin xyz="0 0 0" />
+            <geometry>
+                <cylinder radius="0.024" length="0.044" />
+            </geometry>
+        </collision>
+        <xacro:inertial_cylinder mass="0.1" radius="0.024" length="0.044">
+            <origin xyz="0 0 0" rpy="0 0 1" />
+        </xacro:inertial_cylinder>
+    </link>
+    <joint name="wheel_right2_joint" type="continuous">
+        <parent link="chassis" />
+        <child link="right_wheel2" />
+        <axis xyz="0 0 1"/>
+        <origin rpy="${-pi/2} 0 0" xyz="0.005 -0.066 0.0165"/>
+    </joint>
+    <link name="right_wheel2">
+        <visual>
+            <origin xyz="0 0 0" />
+            <geometry>
+                <cylinder radius="0.024" length="0.044" />
+            </geometry>
+            <material name="white" />
+        </visual>
+        <collision>
+            <origin xyz="0 0 0" />
+            <geometry>
+                <cylinder radius="0.024" length="0.044" />
+            </geometry>
+        </collision>
+        <xacro:inertial_cylinder mass="0.1" radius="0.024" length="0.044">
+            <origin xyz="0 0 0" rpy="0 0 1" />
+        </xacro:inertial_cylinder>
+    </link>
+    <joint name="wheel_right3_joint" type="continuous">
+        <parent link="chassis" />
+        <child link="right_wheel3" />
+        <axis xyz="0 0 1"/>
+        <origin rpy="${-pi/2} 0 0" xyz="-0.055 -0.066 0.0165"/>
+    </joint>
+    <link name="right_wheel3">
+        <visual>
+            <origin xyz="0 0 0" />
+            <geometry>
+                <cylinder radius="0.024" length="0.044" />
+            </geometry>
+            <material name="white" />
+        </visual>
+        <collision>
+            <origin xyz="0 0 0" />
+            <geometry>
+                <cylinder radius="0.024" length="0.044" />
+            </geometry>
+        </collision>
+        <xacro:inertial_cylinder mass="0.1" radius="0.024" length="0.044">
+            <origin xyz="0 0 0" rpy="0 0 1" />
+        </xacro:inertial_cylinder>
+    </link>
+    <!-- EARS -->
+    <joint name="left_ear_joint" type="revolute">
+        <parent link="base" />
+        <child link="left_ear" />
+        <axis xyz="0 1 0"/>
+        <origin rpy="0 0 0" xyz="-0.09 0.075 0.09" />
+        <limit effort="1" velocity="1" upper="${-pi/2}" lower="${pi/4}" />
+    </joint>
+    <link name="left_ear">
+        <visual>
+            <origin xyz="0 0 0" />
+            <geometry>
+                <mesh filename="package://kapibara/meshes/Wing1.stl" scale="0.001 0.001 0.001" />
+            </geometry>
+            <material name="white" />
+        </visual>
+    </link>
+     <joint name="right_ear_joint" type="revolute">
+        <parent link="base" />
+        <child link="righ_ear" />
+        <axis xyz="0 1 0"/>
+        <origin rpy="0 0 0" xyz="-0.09 -0.070 0.09" />
+        <limit effort="1" velocity="1" upper="${-pi/2}" lower="${pi/4}" />
+    </joint>
+    <link name="righ_ear">
+        <visual>
+            <origin xyz="0 0 0" />
+            <geometry>
+                <mesh filename="package://kapibara/meshes/Wing2.stl" scale="0.001 0.001 0.001" />
+            </geometry>
+            <material name="white" />
+        </visual>
     </link>
 </robot>

Commit message: I have fixed collisions in URDF

File: src/workspace/src/kapibara/description/robot_core.xacro (robot description, xacro)
@@ -29,5 +29,5 @@
         </visual>
         <collision>
-            <origin xyz="0 0 0" />
+            <origin xyz="0 0 0.02" />
             <geometry>
                 <box size="0.150 0.083 0.033" />
@@ -35,7 +35,10 @@
         </collision>
         <xacro:inertial_box mass="0.65" x="0.15" y="0.083" z="0.033" >
-            <origin xyz="0 0 0" rpy="0 0 0" />
+            <origin xyz="0 0 0.02" rpy="0 0 0" />
         </xacro:inertial_box>
     </link>
+    <gazebo reference="chassis">
+        <material>Gazebo/Black</material>
+    </gazebo>
     <!-- Base -->
     <joint name="base_joint" type="fixed">
@@ -53,5 +56,5 @@
         </visual>
         <collision>
-            <origin xyz="0 0 0.05" />
+            <origin xyz="-0.02 0 0.07" />
             <geometry>
                 <box size="0.279 0.134 0.161" />
@@ -59,7 +62,10 @@
         </collision>
         <xacro:inertial_box mass="1.15" x="0.279" y="0.134" z="0.161" >
-            <origin xyz="0 0 0.05" rpy="0 0 0" />
+            <origin xyz="-0.02 0 0.07" rpy="0 0 0" />
         </xacro:inertial_box>
     </link>
+    <gazebo reference="base">
+        <material>Gazebo/Orange</material>
+    </gazebo>
     <!-- LEFT WHEEL LINK -->
     <joint name="wheel_left1_joint" type="continuous">
