Commit message: I have added laser distance sensors

File: src/workspace/src/kapibara/description/camera.xacro (robot description, xacro)
@@ -40,4 +40,8 @@
             </camera>
             <plugin name="camera_controller" filename="libgazebo_ros_camera.so">
+                <ros>
+                <namespace>KapiBara</namespace>
+                <remapping>~/out:=camera</remapping>
+                </ros>
                 <frame_name>camera_link_optical</frame_name>
             </plugin>

File: src/workspace/src/kapibara/description/kapibara.urdf.xacro (robot description, xacro)
@@ -2,6 +2,7 @@
 <robot xmlns:xacro="http://www.ros.org/wiki/xacro" name="robot">
     <xacro:include filename="robot_core.xacro" />
-    <xacro:include filename="ros2_control.xacro" />
     <xacro:include filename="camera.xacro" />
+    <xacro:include filename="lasers_joints.xacro" />
+    <!-- <xacro:include filename="ros2_control.xacro" /> -->
     <!-- <xacro:include filename="gazebo control.xacro" /> -->
 </robot>

File: src/workspace/src/kapibara/description/robot_core.xacro (robot description, xacro)
@@ -10,4 +10,7 @@
     <material name="black">
         <color rgba="0 0 0 1" />
+    </material>
+    <material name="red">
+        <color rgba="1 0 0 1" />
     </material>
     <!-- BASE LINK -->
