Commit message: Changes to URDF model

File: src/workspace/src/kapibara/description/kapibara.urdf.xacro (robot description, xacro)
@@ -1,6 +1,6 @@
 <?xml version="1.0"?>
 <robot xmlns:xacro="http://www.ros.org/wiki/xacro" name="robot">
-    <xacro:include filename="robot_core.xacro"/>
-    <xacro:include filename="ros2_control.xacro"/>
+    <xacro:include filename="robot_core.xacro" />
+    <xacro:include filename="ros2_control.xacro" />
     <!-- <xacro:include filename="gazebo control.xacro" /> -->
 </robot>

File: src/workspace/src/kapibara/description/robot_core.xacro (robot description, xacro)
@@ -58,8 +58,8 @@
             <origin xyz="-0.02 0 0.07" />
             <geometry>
-                <box size="0.279 0.134 0.161" />
-            </geometry>
-        </collision>
-        <xacro:inertial_box mass="1.15" x="0.279" y="0.134" z="0.161" >
+                <box size="0.279 0.134 0.15" />
+            </geometry>
+        </collision>
+        <xacro:inertial_box mass="1.15" x="0.279" y="0.134" z="0.15" >
             <origin xyz="-0.02 0 0.07" rpy="0 0 0" />
         </xacro:inertial_box>

File: src/workspace/src/kapibara/description/ros2_control.xacro (robot description, xacro)
@@ -6,4 +6,20 @@
         </hardware>
         <joint name="wheel_left1_joint">
+            <command_interface name="velocity">
+                <param name="min">-10</param>
+                <param name="max">10</param>
+            </command_interface>
+            <state_interface name="velocity" />
+            <state_interface name="position" />
+        </joint>
+        <joint name="wheel_left2_joint">
+            <command_interface name="velocity">
+                <param name="min">-10</param>
+                <param name="max">10</param>
+            </command_interface>
+            <state_interface name="velocity" />
+            <state_interface name="position" />
+        </joint>
+        <joint name="wheel_left3_joint">
             <command_interface name="velocity">
                 <param name="min">-10</param>
@@ -21,4 +37,20 @@
             <state_interface name="position" />
         </joint>
+        <joint name="wheel_right2_joint">
+            <command_interface name="velocity">
+                <param name="min">-10</param>
+                <param name="max">10</param>
+            </command_interface>
+            <state_interface name="velocity" />
+            <state_interface name="position" />
+        </joint>
+        <joint name="wheel_right1_joint">
+            <command_interface name="velocity">
+                <param name="min">-10</param>
+                <param name="max">10</param>
+            </command_interface>
+            <state_interface name="velocity" />
+            <state_interface name="position" />
+        </joint>
     </ros2_control>
     <gazebo>

Commit message: I have fucked up because of my own stupidity but now everything is fine, now gazebo is using GPU so it works quite smoothly

File: src/workspace/src/kapibara/description/kapibara.urdf.xacro (robot description, xacro)
@@ -3,4 +3,5 @@
     <xacro:include filename="robot_core.xacro" />
     <xacro:include filename="ros2_control.xacro" />
+    <xacro:include filename="camera.xacro" />
     <!-- <xacro:include filename="gazebo control.xacro" /> -->
 </robot>

File: src/workspace/src/kapibara/description/robot_core.xacro (robot description, xacro)
@@ -24,5 +24,5 @@
             <origin xyz="0 0 0" />
             <geometry>
-                <mesh filename="package://kapibara/meshes/Bottom.stl" scale="0.001 0.001 0.001" />
+                <mesh filename="file://$(find kapibara)/meshes/Bottom.stl" scale="0.001 0.001 0.001" />
             </geometry>
             <material name="black" />
@@ -51,5 +51,5 @@
             <origin xyz="0 0 0.05" />
             <geometry>
-                <mesh filename="package://kapibara/meshes/Top.stl" scale="0.001 0.001 0.001" />
+                <mesh filename="file://$(find kapibara)/meshes/Top.stl" scale="0.001 0.001 0.001" />
             </geometry>
             <material name="orange" />

Commit message: I have added most of sensors to 3d model, I still need to figure out how to simulate microphones, and the communication layers, after all I am going to use it with standarized protobuf communication layer

File: src/workspace/src/kapibara/description/kapibara.urdf.xacro (robot description, xacro)
@@ -4,4 +4,5 @@
     <xacro:include filename="camera.xacro" />
     <xacro:include filename="lasers_joints.xacro" />
+    <xacro:include filename="imu.xacro" />
     <!-- <xacro:include filename="ros2_control.xacro" /> -->
     <!-- <xacro:include filename="gazebo control.xacro" /> -->

File: src/workspace/src/kapibara/description/robot_core.xacro (robot description, xacro)
@@ -222,6 +222,6 @@
         <child link="left_ear" />
         <axis xyz="0 1 0"/>
-        <origin rpy="0 0 0" xyz="-0.09 0.075 0.09" />
-        <limit effort="1" velocity="1" upper="${-pi/2}" lower="${pi/4}" />
+        <origin rpy="0 ${-pi/2} 0" xyz="-0.09 0.075 0.09" />
+        <limit effort="1" velocity="1" upper="${pi}" lower="0" />
     </joint>
     <link name="left_ear">
@@ -233,4 +233,13 @@
             <material name="white" />
         </visual>
+        <collision>
+            <origin xyz="0 0 0" rpy="${pi/2} 0 0"/>
+            <geometry>
+                <cylinder radius="0.024" length="0.01" />
+            </geometry>
+        </collision>
+        <xacro:inertial_cylinder mass="0.1" radius="0.024" length="0.01">
+            <origin xyz="0 0 0" rpy="${pi/2} 0 0" />
+        </xacro:inertial_cylinder>
     </link>
      <joint name="right_ear_joint" type="revolute">
@@ -238,6 +247,6 @@
         <child link="righ_ear" />
         <axis xyz="0 1 0"/>
-        <origin rpy="0 0 0" xyz="-0.09 -0.070 0.09" />
-        <limit effort="1" velocity="1" upper="${-pi/2}" lower="${pi/4}" />
+        <origin rpy="0 ${-pi/2} 0" xyz="-0.09 -0.070 0.09" />
+        <limit effort="1" velocity="1" upper="${pi}" lower="0" />
     </joint>
     <link name="righ_ear">
@@ -249,4 +258,13 @@
             <material name="white" />
         </visual>
+        <collision>
+            <origin xyz="0 0 0" rpy="${pi/2} 0 0" />
+            <geometry>
+                <cylinder radius="0.024" length="0.01" />
+            </geometry>
+        </collision>
+        <xacro:inertial_cylinder mass="0.1" radius="0.024" length="0.01">
+            <origin xyz="0 0 0" rpy="${pi/2} 0 0" />
+        </xacro:inertial_cylinder>
     </link>
 </robot>
