Commit message: Now it working I cannot set namespace for controller manager so I will just use simple remap, I won't be using multiple KapiBaras in one Gazebo simulation afterall, for now...

File: gazebo/src/workspace/src/kapibara/description/kapibara.urdf.xacro (robot description, xacro)
@@ -5,5 +5,5 @@
     <xacro:include filename="lasers_joints.xacro" />
     <xacro:include filename="imu.xacro" />
-    <!-- <xacro:include filename="ros2_control.xacro" /> -->
+    <xacro:include filename="ros2_control.xacro" />
     <!-- <xacro:include filename="gazebo control.xacro" /> -->
 </robot>

File: gazebo/src/workspace/src/kapibara/description/ros2_control.xacro (robot description, xacro)
@@ -6,20 +6,4 @@
         </hardware>
         <joint name="wheel_left1_joint">
-            <command_interface name="velocity">
-                <param name="min">-10</param>
-                <param name="max">10</param>
-            </command_interface>
-            <state_interface name="velocity" />
-            <state_interface name="position" />
-        </joint>
-        <joint name="wheel_left2_joint">
-            <command_interface name="velocity">
-                <param name="min">-10</param>
-                <param name="max">10</param>
-            </command_interface>
-            <state_interface name="velocity" />
-            <state_interface name="position" />
-        </joint>
-        <joint name="wheel_left3_joint">
             <command_interface name="velocity">
                 <param name="min">-10</param>
@@ -37,24 +21,11 @@
             <state_interface name="position" />
         </joint>
-        <joint name="wheel_right2_joint">
-            <command_interface name="velocity">
-                <param name="min">-10</param>
-                <param name="max">10</param>
-            </command_interface>
-            <state_interface name="velocity" />
-            <state_interface name="position" />
-        </joint>
-        <joint name="wheel_right1_joint">
-            <command_interface name="velocity">
-                <param name="min">-10</param>
-                <param name="max">10</param>
-            </command_interface>
-            <state_interface name="velocity" />
-            <state_interface name="position" />
-        </joint>
     </ros2_control>
     <gazebo>
         <plugin name="gazebo_ros2_control" filename="libgazebo_ros2_control.so">
             <parameters>$(find kapibara)/config/my_controllers.yaml</parameters>
+             <!--<ros>
+                <namespace>KapiBara</namespace>
+            </ros>-->
         </plugin>
     </gazebo>
