Commit message: I have made robot to work with real hardware, now I need to write proper hardware interface

File: gazebo/src/workspace/src/kapibara/description/imu.xacro (robot description, xacro)
@@ -56,5 +56,5 @@
         <plugin name="kapibara_imu" filename="libgazebo_ros_imu_sensor.so">
             <ros>
-                <namespace>KapiBara</namespace>
+                <namespace>Gazebo</namespace>
                 <remapping>~/out:=imu</remapping>
             </ros>

File: gazebo/src/workspace/src/kapibara/description/kapibara.urdf.xacro (robot description, xacro)
@@ -1,4 +1,5 @@
 <?xml version="1.0"?>
 <robot xmlns:xacro="http://www.ros.org/wiki/xacro" name="robot">
+    <xacro:arg name="sim_mode" default="false"/>
     <xacro:include filename="robot_core.xacro" />
     <xacro:include filename="camera.xacro" />

File: gazebo/src/workspace/src/kapibara/description/lasers_def.xacro (robot description, xacro)
@@ -37,5 +37,5 @@
             <plugin name="${sensor_name}_laserscan" filename="libgazebo_ros_ray_sensor.so">
                 <ros>
-                <namespace>KapiBara</namespace>
+                <namespace>Gazebo</namespace>
                 <remapping>~/out:=${sensor_name}</remapping>
                 </ros>

File: gazebo/src/workspace/src/kapibara/description/ros2_control.xacro (robot description, xacro)
@@ -1,31 +1,54 @@
 <?xml version="1.0"?>
 <robot xmlns:xacro="http://www.ros.org/wiki/xacro">
-    <ros2_control name="GazeboSystem" type="system">
-        <hardware>
-            <plugin>gazebo_ros2_control/GazeboSystem</plugin>
-        </hardware>
-        <joint name="wheel_left1_joint">
-            <command_interface name="velocity">
-                <param name="min">-10</param>
-                <param name="max">10</param>
-            </command_interface>
-            <state_interface name="velocity" />
-            <state_interface name="position" />
-        </joint>
-        <joint name="wheel_right3_joint">
-            <command_interface name="velocity">
-                <param name="min">-10</param>
-                <param name="max">10</param>
-            </command_interface>
-            <state_interface name="velocity" />
-            <state_interface name="position" />
-        </joint>
-    </ros2_control>
+    <xacro:unless value="${arg sim_mode}">
+        <ros2_control name="KapiBaraMotors" type="system">
+            <hardware>
+                <plugin>kapibara/MotorDriver</plugin>
+            </hardware>
+            <joint name="wheel_left1_joint">
+                <command_interface name="velocity">
+                    <param name="min">-10</param>
+                    <param name="max">10</param>
+                </command_interface>
+                <state_interface name="velocity" />
+                <state_interface name="position" />
+            </joint>
+            <joint name="wheel_right3_joint">
+                <command_interface name="velocity">
+                    <param name="min">-10</param>
+                    <param name="max">10</param>
+                </command_interface>
+                <state_interface name="velocity" />
+                <state_interface name="position" />
+            </joint>
+        </ros2_control>
+    </xacro:unless>
+    <xacro:if value="${arg sim_mode}">
+        <ros2_control name="GazeboSystem" type="system">
+            <hardware>
+                <plugin>gazebo_ros2_control/GazeboSystem</plugin>
+            </hardware>
+            <joint name="wheel_left1_joint">
+                <command_interface name="velocity">
+                    <param name="min">-10</param>
+                    <param name="max">10</param>
+                </command_interface>
+                <state_interface name="velocity" />
+                <state_interface name="position" />
+            </joint>
+            <joint name="wheel_right3_joint">
+                <command_interface name="velocity">
+                    <param name="min">-10</param>
+                    <param name="max">10</param>
+                </command_interface>
+                <state_interface name="velocity" />
+                <state_interface name="position" />
+            </joint>
+        </ros2_control>
+    </xacro:if>
     <gazebo>
         <plugin name="gazebo_ros2_control" filename="libgazebo_ros2_control.so">
             <parameters>$(find kapibara)/config/my_controllers.yaml</parameters>
-             <!--<ros>
-                <namespace>KapiBara</namespace>
-            </ros>-->
+            <parameters>$(find kapibara)/config/my_controllers_sim.yaml</parameters>
         </plugin>
     </gazebo>
