Commit message: I have fixed ears orientation

File: gazebo/src/workspace/src/kapibara/description/robot_core.xacro (robot description, xacro)
@@ -221,6 +221,6 @@
         <parent link="base" />
         <child link="left_ear" />
-        <axis xyz="0 1 0"/>
-        <origin rpy="0 ${-pi/2} 0" xyz="-0.09 0.075 0.09" />
+        <axis xyz="0 -1 0"/>
+        <origin rpy="0 ${pi/2} 0" xyz="-0.09 0.075 0.09" />
         <limit effort="1" velocity="1" upper="${pi}" lower="0" />
     </joint>
@@ -246,6 +246,6 @@
         <parent link="base" />
         <child link="righ_ear" />
-        <axis xyz="0 1 0"/>
-        <origin rpy="0 ${-pi/2} 0" xyz="-0.09 -0.070 0.09" />
+        <axis xyz="0 -1 0"/>
+        <origin rpy="0 ${pi/2} 0" xyz="-0.09 -0.070 0.09" />
         <limit effort="1" velocity="1" upper="${pi}" lower="0" />
     </joint>

Commit message: I am almost fixed KapiBara URDF

File: gazebo/src/workspace/src/kapibara/description/robot_core.xacro (robot description, xacro)
@@ -31,13 +31,96 @@
             <material name="black" />
         </visual>
-        <collision>
-            <origin xyz="0 0 0.02" />
-            <geometry>
-                <box size="0.150 0.083 0.033" />
-            </geometry>
-        </collision>
-        <xacro:inertial_box mass="0.65" x="0.15" y="0.083" z="0.033" >
-            <origin xyz="0 0 0.02" rpy="0 0 0" />
-        </xacro:inertial_box>
+        <visual name="left_wheel2_visual">
+            <origin rpy="${-pi/2} 0 0" xyz="0.065 0.066 0.01"/>
+            <geometry>
+                <cylinder radius="0.024" length="0.044" />
+            </geometry>
+            <material name="white" />
+        </visual>
+        <collision name="left_wheel2_collision">
+            <origin rpy="${-pi/2} 0 0" xyz="0.065 0.066 0.01"/>
+            <geometry>
+                <cylinder radius="0.024" length="0.044" />
+            </geometry>
+            <surface>
+                <friction>
+                    <ode>
+                    <mu>0</mu>
+                    <mu2>0</mu2>
+                    <slip1>1.0</slip1>
+                    <slip2>1.0</slip2>
+                    </ode>
+                </friction>
+            </surface>
+        </collision>
+        <visual name="left_wheel3_visual">
+            <origin rpy="${-pi/2} 0 0" xyz="-0.055 0.066 0.01"/>
+            <geometry>
+                <cylinder radius="0.024" length="0.044" />
+            </geometry>
+            <material name="white" />
+        </visual>
+        <collision name="left_wheel3_collision">
+            <origin rpy="${-pi/2} 0 0" xyz="-0.055 0.066 0.01"/>
+            <geometry>
+                <cylinder radius="0.024" length="0.044" />
+            </geometry>
+            <surface>
+                <friction>
+                    <ode>
+                    <mu>0</mu>
+                    <mu2>0</mu2>
+                    <slip1>1.0</slip1>
+                    <slip2>1.0</slip2>
+                    </ode>
+                </friction>
+            </surface>
+        </collision>
+        <visual name="right_wheel2_visual">
+            <origin rpy="${-pi/2} 0 0" xyz="0.065 -0.066 0.01"/>
+            <geometry>
+                <cylinder radius="0.024" length="0.044" />
+            </geometry>
+            <material name="white" />
+        </visual>
+        <collision name="right_wheel2_collision">
+            <origin rpy="${-pi/2} 0 0" xyz="0.065 -0.066 0.01"/>
+            <geometry>
+                <cylinder radius="0.024" length="0.044" />
+            </geometry>
+            <surface>
+                <friction>
+                    <ode>
+                    <mu>0</mu>
+                    <mu2>0</mu2>
+                    <slip1>1.0</slip1>
+                    <slip2>1.0</slip2>
+                    </ode>
+                </friction>
+            </surface>
+        </collision>
+        <visual name="right_wheel3_visual">
+            <origin rpy="${-pi/2} 0 0" xyz="-0.055 -0.066 0.01"/>
+            <geometry>
+                <cylinder radius="0.024" length="0.044" />
+            </geometry>
+            <material name="white" />
+        </visual>
+        <collision name="right_wheel3_collision">
+            <origin rpy="${-pi/2} 0 0" xyz="-0.055 -0.066 0.01"/>
+            <geometry>
+                <cylinder radius="0.024" length="0.044" />
+            </geometry>
+            <surface>
+                <friction>
+                    <ode>
+                    <mu>0</mu>
+                    <mu2>0</mu2>
+                    <slip1>1.0</slip1>
+                    <slip2>1.0</slip2>
+                    </ode>
+                </friction>
+            </surface>
+        </collision>
     </link>
     <gazebo reference="chassis">
@@ -76,5 +159,7 @@
         <child link="left_wheel1" />
         <axis xyz="0 0 1"/>
-        <origin rpy="${-pi/2} 0 0" xyz="0.065 0.066 0.0165"/>
+        <origin rpy="${-pi/2} 0 0" xyz="0.005 0.066 0.01"/>
+        <joint_properties damping="1.0" friction="1.0" />
+        <!-- <limit effort="10000" velocity="1000"/>  -->
     </joint>
     <link name="left_wheel1">
@@ -96,9 +181,10 @@
         </xacro:inertial_cylinder>
     </link>
-    <joint name="wheel_left2_joint" type="continuous">
+    <!-- <joint name="wheel_left2_joint" type="continuous">
         <parent link="chassis" />
         <child link="left_wheel2" />
         <axis xyz="0 0 1"/>
         <origin rpy="${-pi/2} 0 0" xyz="0.005 0.066 0.0165"/>
+        <joint_properties damping="1.0" friction="1.0" />
     </joint>
     <link name="left_wheel2">
@@ -125,4 +211,5 @@
         <axis xyz="0 0 1"/>
         <origin rpy="${-pi/2} 0 0" xyz="-0.055 0.066 0.0165"/>
+        <joint_properties damping="1.0" friction="1.0" />
     </joint>
     <link name="left_wheel3">
@@ -143,5 +230,5 @@
             <origin xyz="0 0 0" rpy="0 0 1" />
         </xacro:inertial_cylinder>
-    </link>
+    </link> -->
     <!-- RIGHT WHEEL LINK -->
     <joint name="wheel_right1_joint" type="continuous">
@@ -149,5 +236,7 @@
         <child link="right_wheel1" />
         <axis xyz="0 0 1"/>
-        <origin rpy="${-pi/2} 0 0" xyz="0.065 -0.066 0.0165"/>
+        <origin rpy="${-pi/2} 0 0" xyz="0.005 -0.066 0.01"/>
+        <joint_properties damping="1.0" friction="1.0" />
+        <!-- <limit effort="10000" velocity="1000"/>  -->
     </joint>
     <link name="right_wheel1">
@@ -169,9 +258,10 @@
         </xacro:inertial_cylinder>
     </link>
-    <joint name="wheel_right2_joint" type="continuous">
+    <!-- <joint name="wheel_right2_joint" type="continuous">
         <parent link="chassis" />
         <child link="right_wheel2" />
         <axis xyz="0 0 1"/>
         <origin rpy="${-pi/2} 0 0" xyz="0.005 -0.066 0.0165"/>
+        <joint_properties damping="1.0" friction="1.0" />
     </joint>
     <link name="right_wheel2">
@@ -198,4 +288,5 @@
         <axis xyz="0 0 1"/>
         <origin rpy="${-pi/2} 0 0" xyz="-0.055 -0.066 0.0165"/>
+        <joint_properties damping="1.0" friction="1.0" />
     </joint>
     <link name="right_wheel3">
@@ -216,5 +307,5 @@
             <origin xyz="0 0 0" rpy="0 0 1" />
         </xacro:inertial_cylinder>
-    </link>
+    </link> -->
     <!-- EARS -->
     <joint name="left_ear_joint" type="revolute">

File: gazebo/src/workspace/src/kapibara/description/ros2_control.xacro (robot description, xacro)
@@ -6,5 +6,5 @@
                 <plugin>tb6612_drive_simple/TB6612DriveSimple</plugin>
                 <param name="left_wheel_name">wheel_left1_joint</param>
-                <param name="right_wheel_name">wheel_right3_joint</param>
+                <param name="right_wheel_name">wheel_right1_joint</param>
                 <param name="max_speed">10</param>
                 <param name="loop_rate">30</param>
@@ -22,5 +22,5 @@
                 <state_interface name="position" />
             </joint>
-            <joint name="wheel_right3_joint">
+            <joint name="wheel_right1_joint">
                 <command_interface name="velocity">
                     <param name="min">-10</param>
@@ -45,5 +45,5 @@
                 <state_interface name="position" />
             </joint>
-            <joint name="wheel_right3_joint">
+            <joint name="wheel_right1_joint">
                 <command_interface name="velocity">
                     <param name="min">-10</param>

Commit message: I think I have fixed it is perfectly circing around

File: gazebo/src/workspace/src/kapibara/description/robot_core.xacro (robot description, xacro)
@@ -31,5 +31,5 @@
             <material name="black" />
         </visual>
-        <visual name="left_wheel2_visual">
+        <!-- <visual name="left_wheel2_visual">
             <origin rpy="${-pi/2} 0 0" xyz="0.065 0.066 0.01"/>
             <geometry>
@@ -122,5 +122,5 @@
                 </friction>
             </surface>
-        </collision>
+        </collision> -->
     </link>
     <gazebo reference="chassis">
@@ -159,5 +159,5 @@
         <child link="left_wheel1" />
         <axis xyz="0 0 1"/>
-        <origin rpy="${-pi/2} 0 0" xyz="0.005 0.066 0.01"/>
+        <origin rpy="${-pi/2} 0 0" xyz="0.005 0.066 0.0135"/>
         <joint_properties damping="1.0" friction="1.0" />
         <!-- <limit effort="10000" velocity="1000"/>  -->
@@ -181,10 +181,9 @@
         </xacro:inertial_cylinder>
     </link>
-    <!-- <joint name="wheel_left2_joint" type="continuous">
+    <joint name="wheel_left2_joint" type="fixed">
         <parent link="chassis" />
         <child link="left_wheel2" />
         <axis xyz="0 0 1"/>
-        <origin rpy="${-pi/2} 0 0" xyz="0.005 0.066 0.0165"/>
-        <joint_properties damping="1.0" friction="1.0" />
+        <origin rpy="${-pi/2} 0 0" xyz="0.065 0.066 0.0135"/>
     </joint>
     <link name="left_wheel2">
@@ -206,10 +205,14 @@
         </xacro:inertial_cylinder>
     </link>
-    <joint name="wheel_left3_joint" type="continuous">
+    <gazebo reference="left_wheel2">
+        <material>Gazebo/White</material>
+        <mu1 value="0.001"/>
+        <mu2 value="0.001"/>
+    </gazebo>
+    <joint name="wheel_left3_joint" type="fixed">
         <parent link="chassis" />
         <child link="left_wheel3" />
         <axis xyz="0 0 1"/>
-        <origin rpy="${-pi/2} 0 0" xyz="-0.055 0.066 0.0165"/>
-        <joint_properties damping="1.0" friction="1.0" />
+        <origin rpy="${-pi/2} 0 0" xyz="-0.055 0.066 0.0135"/>
     </joint>
     <link name="left_wheel3">
@@ -230,5 +233,10 @@
             <origin xyz="0 0 0" rpy="0 0 1" />
         </xacro:inertial_cylinder>
-    </link> -->
+    </link>
+    <gazebo reference="left_wheel3">
+        <material>Gazebo/White</material>
+        <mu1 value="0.001"/>
+        <mu2 value="0.001"/>
+    </gazebo>
     <!-- RIGHT WHEEL LINK -->
     <joint name="wheel_right1_joint" type="continuous">
@@ -236,5 +244,5 @@
         <child link="right_wheel1" />
         <axis xyz="0 0 1"/>
-        <origin rpy="${-pi/2} 0 0" xyz="0.005 -0.066 0.01"/>
+        <origin rpy="${-pi/2} 0 0" xyz="0.005 -0.066 0.0135"/>
         <joint_properties damping="1.0" friction="1.0" />
         <!-- <limit effort="10000" velocity="1000"/>  -->
@@ -258,10 +266,9 @@
         </xacro:inertial_cylinder>
     </link>
-    <!-- <joint name="wheel_right2_joint" type="continuous">
+    <joint name="wheel_right2_joint" type="fixed">
         <parent link="chassis" />
         <child link="right_wheel2" />
         <axis xyz="0 0 1"/>
-        <origin rpy="${-pi/2} 0 0" xyz="0.005 -0.066 0.0165"/>
-        <joint_properties damping="1.0" friction="1.0" />
+        <origin rpy="${-pi/2} 0 0" xyz="0.065 -0.066 0.0135"/>
     </joint>
     <link name="right_wheel2">
@@ -283,10 +290,14 @@
         </xacro:inertial_cylinder>
     </link>
-    <joint name="wheel_right3_joint" type="continuous">
+    <gazebo reference="right_wheel2">
+        <material>Gazebo/White</material>
+        <mu1 value="0.001"/>
+        <mu2 value="0.001"/>
+    </gazebo>
+    <joint name="wheel_right3_joint" type="fixed">
         <parent link="chassis" />
         <child link="right_wheel3" />
         <axis xyz="0 0 1"/>
-        <origin rpy="${-pi/2} 0 0" xyz="-0.055 -0.066 0.0165"/>
-        <joint_properties damping="1.0" friction="1.0" />
+        <origin rpy="${-pi/2} 0 0" xyz="-0.055 -0.066 0.0135"/>
     </joint>
     <link name="right_wheel3">
@@ -307,5 +318,10 @@
             <origin xyz="0 0 0" rpy="0 0 1" />
         </xacro:inertial_cylinder>
-    </link> -->
+    </link>
+    <gazebo reference="right_wheel3">
+        <material>Gazebo/White</material>
+        <mu1 value="0.001"/>
+        <mu2 value="0.001"/>
+    </gazebo>
     <!-- EARS -->
     <joint name="left_ear_joint" type="revolute">

Commit message: It moves forward but It struggle to rotate

File: gazebo/src/workspace/src/kapibara/description/robot_core.xacro (robot description, xacro)
@@ -31,96 +31,4 @@
             <material name="black" />
         </visual>
-        <!-- <visual name="left_wheel2_visual">
-            <origin rpy="${-pi/2} 0 0" xyz="0.065 0.066 0.01"/>
-            <geometry>
-                <cylinder radius="0.024" length="0.044" />
-            </geometry>
-            <material name="white" />
-        </visual>
-        <collision name="left_wheel2_collision">
-            <origin rpy="${-pi/2} 0 0" xyz="0.065 0.066 0.01"/>
-            <geometry>
-                <cylinder radius="0.024" length="0.044" />
-            </geometry>
-            <surface>
-                <friction>
-                    <ode>
-                    <mu>0</mu>
-                    <mu2>0</mu2>
-                    <slip1>1.0</slip1>
-                    <slip2>1.0</slip2>
-                    </ode>
-                </friction>
-            </surface>
-        </collision>
-        <visual name="left_wheel3_visual">
-            <origin rpy="${-pi/2} 0 0" xyz="-0.055 0.066 0.01"/>
-            <geometry>
-                <cylinder radius="0.024" length="0.044" />
-            </geometry>
-            <material name="white" />
-        </visual>
-        <collision name="left_wheel3_collision">
-            <origin rpy="${-pi/2} 0 0" xyz="-0.055 0.066 0.01"/>
-            <geometry>
-                <cylinder radius="0.024" length="0.044" />
-            </geometry>
-            <surface>
-                <friction>
-                    <ode>
-                    <mu>0</mu>
-                    <mu2>0</mu2>
-                    <slip1>1.0</slip1>
-                    <slip2>1.0</slip2>
-                    </ode>
-                </friction>
-            </surface>
-        </collision>
-        <visual name="right_wheel2_visual">
-            <origin rpy="${-pi/2} 0 0" xyz="0.065 -0.066 0.01"/>
-            <geometry>
-                <cylinder radius="0.024" length="0.044" />
-            </geometry>
-            <material name="white" />
-        </visual>
-        <collision name="right_wheel2_collision">
-            <origin rpy="${-pi/2} 0 0" xyz="0.065 -0.066 0.01"/>
-            <geometry>
-                <cylinder radius="0.024" length="0.044" />
-            </geometry>
-            <surface>
-                <friction>
-                    <ode>
-                    <mu>0</mu>
-                    <mu2>0</mu2>
-                    <slip1>1.0</slip1>
-                    <slip2>1.0</slip2>
-                    </ode>
-                </friction>
-            </surface>
-        </collision>
-        <visual name="right_wheel3_visual">
-            <origin rpy="${-pi/2} 0 0" xyz="-0.055 -0.066 0.01"/>
-            <geometry>
-                <cylinder radius="0.024" length="0.044" />
-            </geometry>
-            <material name="white" />
-        </visual>
-        <collision name="right_wheel3_collision">
-            <origin rpy="${-pi/2} 0 0" xyz="-0.055 -0.066 0.01"/>
-            <geometry>
-                <cylinder radius="0.024" length="0.044" />
-            </geometry>
-            <surface>
-                <friction>
-                    <ode>
-                    <mu>0</mu>
-                    <mu2>0</mu2>
-                    <slip1>1.0</slip1>
-                    <slip2>1.0</slip2>
-                    </ode>
-                </friction>
-            </surface>
-        </collision> -->
     </link>
     <gazebo reference="chassis">
@@ -160,5 +68,5 @@
         <axis xyz="0 0 1"/>
         <origin rpy="${-pi/2} 0 0" xyz="0.005 0.066 0.0135"/>
-        <joint_properties damping="1.0" friction="1.0" />
+        <!-- <joint_properties damping="1.0" friction="1.0" />  -->
         <!-- <limit effort="10000" velocity="1000"/>  -->
     </joint>
@@ -181,5 +89,8 @@
         </xacro:inertial_cylinder>
     </link>
-    <joint name="wheel_left2_joint" type="fixed">
+    <gazebo reference="left_wheel1">
+        <material>Gazebo/White</material>
+    </gazebo>
+    <joint name="wheel_left2_joint" type="continuous">
         <parent link="chassis" />
         <child link="left_wheel2" />
@@ -207,8 +118,8 @@
     <gazebo reference="left_wheel2">
         <material>Gazebo/White</material>
-        <mu1 value="0.001"/>
-        <mu2 value="0.001"/>
-    </gazebo>
-    <joint name="wheel_left3_joint" type="fixed">
+        <!-- <mu1 value="0.0001"/> -->
+        <!-- <mu2 value="0.0001"/> -->
+    </gazebo>
+    <joint name="wheel_left3_joint" type="continuous">
         <parent link="chassis" />
         <child link="left_wheel3" />
@@ -236,6 +147,6 @@
     <gazebo reference="left_wheel3">
         <material>Gazebo/White</material>
-        <mu1 value="0.001"/>
-        <mu2 value="0.001"/>
+        <!-- <mu1 value="0.0001"/> -->
+        <!-- <mu2 value="0.0001"/> -->
     </gazebo>
     <!-- RIGHT WHEEL LINK -->
@@ -245,5 +156,5 @@
         <axis xyz="0 0 1"/>
         <origin rpy="${-pi/2} 0 0" xyz="0.005 -0.066 0.0135"/>
-        <joint_properties damping="1.0" friction="1.0" />
+        <!-- <joint_properties damping="1.0" friction="1.0" />  -->
         <!-- <limit effort="10000" velocity="1000"/>  -->
     </joint>
@@ -266,5 +177,8 @@
         </xacro:inertial_cylinder>
     </link>
-    <joint name="wheel_right2_joint" type="fixed">
+    <gazebo reference="right_wheel1">
+        <material>Gazebo/White</material>
+    </gazebo>
+    <joint name="wheel_right2_joint" type="continuous">
         <parent link="chassis" />
         <child link="right_wheel2" />
@@ -292,8 +206,8 @@
     <gazebo reference="right_wheel2">
         <material>Gazebo/White</material>
-        <mu1 value="0.001"/>
-        <mu2 value="0.001"/>
-    </gazebo>
-    <joint name="wheel_right3_joint" type="fixed">
+        <!-- <mu1 value="0.0001"/> -->
+        <!-- <mu2 value="0.0001"/> -->
+    </gazebo>
+    <joint name="wheel_right3_joint" type="continuous">
         <parent link="chassis" />
         <child link="right_wheel3" />
@@ -321,6 +235,6 @@
     <gazebo reference="right_wheel3">
         <material>Gazebo/White</material>
-        <mu1 value="0.001"/>
-        <mu2 value="0.001"/>
+        <!-- <mu1 value="0.0001"/> -->
+        <!-- <mu2 value="0.0001"/> -->
     </gazebo>
     <!-- EARS -->
