Commit message: My robot seems to move forward and rotate correctly

File: gazebo/src/workspace/src/kapibara/description/robot_core.xacro (robot description, xacro)
@@ -86,9 +86,11 @@
         </collision>
         <xacro:inertial_cylinder mass="0.1" radius="0.024" length="0.044">
-            <origin xyz="0 0 0" rpy="0 0 1" />
+            <origin xyz="0 0 0" rpy="0 0 0" />
         </xacro:inertial_cylinder>
     </link>
     <gazebo reference="left_wheel1">
         <material>Gazebo/White</material>
+        <mu1 value="0.1"/>
+        <mu2 value="0.1"/>
     </gazebo>
     <joint name="wheel_left2_joint" type="continuous">
@@ -113,11 +115,11 @@
         </collision>
         <xacro:inertial_cylinder mass="0.1" radius="0.024" length="0.044">
-            <origin xyz="0 0 0" rpy="0 0 1" />
+            <origin xyz="0 0 0" rpy="0 0 0" />
         </xacro:inertial_cylinder>
     </link>
     <gazebo reference="left_wheel2">
         <material>Gazebo/White</material>
-        <!-- <mu1 value="0.0001"/> -->
-        <!-- <mu2 value="0.0001"/> -->
+        <mu1 value="0.1"/>
+        <mu2 value="0.1"/>
     </gazebo>
     <joint name="wheel_left3_joint" type="continuous">
@@ -142,11 +144,11 @@
         </collision>
         <xacro:inertial_cylinder mass="0.1" radius="0.024" length="0.044">
-            <origin xyz="0 0 0" rpy="0 0 1" />
+            <origin xyz="0 0 0" rpy="0 0 0" />
         </xacro:inertial_cylinder>
     </link>
     <gazebo reference="left_wheel3">
         <material>Gazebo/White</material>
-        <!-- <mu1 value="0.0001"/> -->
-        <!-- <mu2 value="0.0001"/> -->
+        <mu1 value="0.1"/>
+        <mu2 value="0.1"/>
     </gazebo>
     <!-- RIGHT WHEEL LINK -->
@@ -174,9 +176,11 @@
         </collision>
         <xacro:inertial_cylinder mass="0.1" radius="0.024" length="0.044">
-            <origin xyz="0 0 0" rpy="0 0 1" />
+            <origin xyz="0 0 0" rpy="0 0 0" />
         </xacro:inertial_cylinder>
     </link>
     <gazebo reference="right_wheel1">
         <material>Gazebo/White</material>
+        <mu1 value="0.1"/>
+        <mu2 value="0.1"/>
     </gazebo>
     <joint name="wheel_right2_joint" type="continuous">
@@ -201,11 +205,11 @@
         </collision>
         <xacro:inertial_cylinder mass="0.1" radius="0.024" length="0.044">
-            <origin xyz="0 0 0" rpy="0 0 1" />
+            <origin xyz="0 0 0" rpy="0 0 0" />
         </xacro:inertial_cylinder>
     </link>
     <gazebo reference="right_wheel2">
         <material>Gazebo/White</material>
-        <!-- <mu1 value="0.0001"/> -->
-        <!-- <mu2 value="0.0001"/> -->
+        <mu1 value="0.1"/>
+        <mu2 value="0.1"/>
     </gazebo>
     <joint name="wheel_right3_joint" type="continuous">
@@ -230,11 +234,11 @@
         </collision>
         <xacro:inertial_cylinder mass="0.1" radius="0.024" length="0.044">
-            <origin xyz="0 0 0" rpy="0 0 1" />
+            <origin xyz="0 0 0" rpy="0 0 0" />
         </xacro:inertial_cylinder>
     </link>
     <gazebo reference="right_wheel3">
         <material>Gazebo/White</material>
-        <!-- <mu1 value="0.0001"/> -->
-        <!-- <mu2 value="0.0001"/> -->
+        <mu1 value="0.1"/>
+        <mu2 value="0.1"/>
     </gazebo>
     <!-- EARS -->

File: gazebo/src/workspace/src/kapibara/description/ros2_control.xacro (robot description, xacro)
@@ -53,4 +53,36 @@
                 <state_interface name="position" />
             </joint>
+            <joint name="wheel_left2_joint">
+                <command_interface name="velocity">
+                    <param name="min">-10</param>
+                    <param name="max">10</param>
+                </command_interface>
+                <state_interface name="velocity" />
+                <state_interface name="position" />
+            </joint>
+            <joint name="wheel_right2_joint">
+                <command_interface name="velocity">
+                    <param name="min">-10</param>
+                    <param name="max">10</param>
+                </command_interface>
+                <state_interface name="velocity" />
+                <state_interface name="position" />
+            </joint>
+            <joint name="wheel_left3_joint">
+                <command_interface name="velocity">
+                    <param name="min">-10</param>
+                    <param name="max">10</param>
+                </command_interface>
+                <state_interface name="velocity" />
+                <state_interface name="position" />
+            </joint>
+            <joint name="wheel_right3_joint">
+                <command_interface name="velocity">
+                    <param name="min">-10</param>
+                    <param name="max">10</param>
+                </command_interface>
+                <state_interface name="velocity" />
+                <state_interface name="position" />
+            </joint>
             <joint name="right_ear_joint">
                 <command_interface name="position">

Commit message: Catch the prey is finished!

File: gazebo/src/workspace/src/kapibara/description/robot_core.xacro (robot description, xacro)
@@ -49,5 +49,5 @@
             <material name="orange" />
         </visual>
-        <collision>
+        <collision name="base_collision">
             <origin xyz="-0.02 0 0.07" />
             <geometry>
@@ -61,4 +61,18 @@
     <gazebo reference="base">
         <material>Gazebo/Orange</material>
+        <sensor type="contact" name="contact_sensor">
+            <always_on>true</always_on>
+            <update_rate>50</update_rate>
+            <contact>
+            <collision>base_link_fixed_joint_lump__base_collision_collision</collision>
+            </contact>
+            <plugin name="bumper_plugin_kapibara" filename="libgazebo_ros_bumper.so">
+                <alwaysOn>true</alwaysOn>
+                <frameName>base</frameName>
+                <ros>
+                <remapping>bumper_states:=collision</remapping>
+                </ros>
+            </plugin>
+      </sensor>
     </gazebo>
     <!-- LEFT WHEEL LINK -->
