Commit message: I am going to make simple maze a bit smaller

File: gazebo/src/workspace/src/kapibara/description/lasers_joints.xacro (robot description, xacro)
@@ -33,5 +33,5 @@
         <parent link="base"/>
         <child link="floor_laser_link"/>
-        <origin xyz="-0.16 0.0 0.021" rpy="0 ${pi/5} ${pi}"/>
+        <origin xyz="0.11 0.0 0.08" rpy="${pi} 0 0"/>
     </joint>
     <link name="floor_laser_link">

Commit message: I have made a bigger maze too!

File: gazebo/src/workspace/src/kapibara/description/lasers_joints.xacro (robot description, xacro)
@@ -33,5 +33,5 @@
         <parent link="base"/>
         <child link="floor_laser_link"/>
-        <origin xyz="0.11 0.0 0.08" rpy="${pi} 0 0"/>
+        <origin xyz="0.11 0.0 0.12" rpy="${pi} 0 0"/>
     </joint>
     <link name="floor_laser_link">

Commit message: I have found some error in Maze but I fixed it and I removed back sensor from KapiBara

File: gazebo/src/workspace/src/kapibara/description/lasers_joints.xacro (robot description, xacro)
@@ -22,18 +22,4 @@
     </joint>
     <link name="front_right_laser_link">
-        <visual>
-            <geometry>
-                <box size="0.01 0.01 0.01" />
-            </geometry>
-            <material name="red" />
-        </visual>
-    </link>
-    <!-- FLOOR DISTANCE SENSOR -->
-    <joint name="floor_laser_joint" type="fixed">
-        <parent link="base"/>
-        <child link="floor_laser_link"/>
-        <origin xyz="0.11 0.0 0.12" rpy="${pi} 0 0"/>
-    </joint>
-    <link name="floor_laser_link">
         <visual>
             <geometry>
@@ -74,5 +60,4 @@
     <xacro:laser_sensor sensor_name="front_left" />
     <xacro:laser_sensor sensor_name="front_right" />
-    <xacro:laser_sensor sensor_name="floor" />
     <xacro:laser_sensor sensor_name="side_left" />
     <xacro:laser_sensor sensor_name="side_right" />
