Commit message: I have mouse model now I am trying to spawn couple of mouse robots

File: gazebo/src/workspace/src/gym/description/mouse.urdf.xacro (robot description, xacro)
@@ -1,14 +1,14 @@
 <?xml version="1.0"?>
-<robot name="differential_drive_robot">
+<robot xmlns:xacro="http://www.ros.org/wiki/xacro" name="mouse_bot">
+  <xacro:arg name="name" default="mouse" />
+  <xacro:include filename="inertial_macros.xacro"/>
   <!-- Link Definitions -->
   <link name="base_link">
-    <inertial>
-      <mass value="1.0"/>
-      <origin xyz="0 0 0" rpy="0 0 0"/>
-      <inertia ixx="0.1" ixy="0.0" ixz="0.0" iyy="0.1" iyz="0.0" izz="0.1"/>
-    </inertial>
+    <xacro:inertial_box mass="1" x="0.5" y="0.5" z="0.5" >
+            <origin xyz="0.0 0 0.0" rpy="0 0 0" />
+        </xacro:inertial_box>
     <visual>
       <geometry>
-        <box size="0.5 0.3 0.1"/>
+        <box size="0.5 0.5 0.5"/>
       </geometry>
       <material name="blue"/>
@@ -16,17 +16,18 @@
     <collision>
       <geometry>
-        <box size="0.5 0.3 0.1"/>
+        <box size="0.5 0.5 0.5"/>
       </geometry>
     </collision>
   </link>
+  <gazebo reference="base_link">
+        <material>Gazebo/Red</material>
+  </gazebo>
   <link name="left_wheel_link">
-    <inertial>
-      <mass value="0.2"/>
-      <origin xyz="0 0 0" rpy="0 0 0"/>
-      <inertia ixx="0.02" ixy="0.0" ixz="0.0" iyy="0.02" iyz="0.0" izz="0.02"/>
-    </inertial>
+    <xacro:inertial_cylinder mass="0.2" radius="0.1" length="0.1">
+        <origin xyz="0 0 0" rpy="0 0 0" />
+    </xacro:inertial_cylinder>
     <visual>
       <geometry>
-        <cylinder length="0.1" radius="0.05"/>
+        <cylinder length="0.1" radius="0.1"/>
       </geometry>
       <material name="black"/>
@@ -34,17 +35,18 @@
     <collision>
       <geometry>
-        <cylinder length="0.1" radius="0.05"/>
+        <cylinder length="0.1" radius="0.1"/>
       </geometry>
     </collision>
   </link>
+  <gazebo reference="left_wheel_link">
+        <material>Gazebo/Black</material>
+  </gazebo>
   <link name="right_wheel_link">
-    <inertial>
-      <mass value="0.2"/>
-      <origin xyz="0 0 0" rpy="0 0 0"/>
-      <inertia ixx="0.02" ixy="0.0" ixz="0.0" iyy="0.02" iyz="0.0" izz="0.02"/>
-    </inertial>
+    <xacro:inertial_cylinder mass="0.2" radius="0.1" length="0.1">
+        <origin xyz="0 0 0" rpy="0 0 0" />
+    </xacro:inertial_cylinder>
     <visual>
       <geometry>
-        <cylinder length="0.1" radius="0.05"/>
+        <cylinder length="0.1" radius="0.1"/>
       </geometry>
       <material name="black"/>
@@ -52,14 +54,15 @@
     <collision>
       <geometry>
-        <cylinder length="0.1" radius="0.05"/>
+        <cylinder length="0.1" radius="0.1"/>
       </geometry>
     </collision>
   </link>
-  <link name="caster_wheel_link">
-    <inertial>
-      <mass value="0.1"/>
-      <origin xyz="0 0 0" rpy="0 0 0"/>
-      <inertia ixx="0.01" ixy="0.0" ixz="0.0" iyy="0.01" iyz="0.0" izz="0.01"/>
-    </inertial>
+  <gazebo reference="right_wheel_link">
+        <material>Gazebo/Black</material>
+  </gazebo>
+  <!-- <link name="caster_wheel_link">
+    <xacro:inertial_sphere mass="0.1" radius="0.05">
+        <origin xyz="0 0 0" rpy="0 0 0" />
+    </xacro:inertial_sphere>
     <visual>
       <geometry>
@@ -73,57 +76,51 @@
       </geometry>
     </collision>
-  </link>
+  </link> -->
+  <gazebo reference="caster_wheel_link">
+        <material>Gazebo/Black</material>
+  </gazebo>
   <!-- Joint Definitions -->
   <joint name="left_wheel_joint" type="continuous">
     <parent link="base_link"/>
     <child link="left_wheel_link"/>
-    <origin xyz="-0.25 0.15 0"/>
-    <axis xyz="0 1 0"/>
+    <origin xyz="-0.25 0.3 -0.15" rpy="${-pi/2} 0 0"/>
+    <axis xyz="0 0 1"/>
   </joint>
   <joint name="right_wheel_joint" type="continuous">
     <parent link="base_link"/>
     <child link="right_wheel_link"/>
-    <origin xyz="-0.25 -0.15 0"/>
-    <axis xyz="0 1 0"/>
+    <origin xyz="-0.25 -0.3 -0.15" rpy="${-pi/2} 0 0"/>
+    <axis xyz="0 0 1"/>
   </joint>
-  <joint name="caster_wheel_joint" type="continuous">
+  <!-- <joint name="caster_wheel_joint" type="continuous">
     <parent link="base_link"/>
     <child link="caster_wheel_link"/>
-    <origin xyz="0.25 0 0"/>
+    <origin xyz="0 0 -0.05"/>
     <axis xyz="0 0 1"/>
-  </joint>
+  </joint> -->
   <!-- ros2_control Configuration -->
-  <ros2_control name="DifferentialDriveController" type="system">
+  <ros2_control name="GazeboSystem" type="system">
     <hardware>
-      <plugin>ros2_control_components/DiffDrive</plugin>
-      <param name="wheel_radius">0.05</param>
-      <param name="track_width">0.3</param>
+      <plugin>gazebo_ros2_control/GazeboSystem</plugin>
+    </hardware>
       <joint name="left_wheel_joint">
-        <param name="motor_command_interface">velocity</param>
-        <param name="state_interface">velocity</param>
+        <command_interface name="velocity" />
+        <state_interface name="velocity" />
+        <state_interface name="position" />
       </joint>
       <joint name="right_wheel_joint">
-        <param name="motor_command_interface">velocity</param>
-        <param name="state_interface">velocity</param>
+        <command_interface name="velocity" />
+        <state_interface name="velocity" />
+        <state_interface name="position" />
       </joint>
-    </hardware>
-    <controller name="mouse_joint_state" type="joint_state_controller/JointStateController">
-      <param name="publish_rate">50</param>
-    </controller>
-    <controller name="mouse_motors" type="diff_drive_controller/DiffDriveController">
-      <param name="left_wheel_names">left_wheel_joint</param>
-      <param name="right_wheel_names">right_wheel_joint</param>
-      <param name="cmd_vel_timeout">0.5</param>
-      <param name="base_frame_id">base_link</param>
-      <param name="odom_frame_id">odom</param>
-      <param name="publish_rate">50</param>
-      <param name="wheel_separation">0.3</param>
-      <param name="wheel_radius">0.05</param>
-    </controller>
   </ros2_control>
   <!-- Gazebo Configuration -->
   <gazebo>
     <plugin name="gazebo_ros2_control" filename="libgazebo_ros2_control.so">
-      <robot_namespace>/</robot_namespace>
+      <ros>
+        <!-- <namespace>/$(arg name)</namespace> -->
+      </ros>
+      <!-- <robot_param_node>/$(arg name)/robot_state_publisher</robot_param_node> -->
+      <parameters>$(find gym)/config/my_controllers.yaml</parameters>
     </plugin>
   </gazebo>

Commit message: Stefan has now a distance sensor

File: gazebo/src/workspace/src/gym/description/mouse.urdf.xacro (robot description, xacro)
@@ -93,4 +93,19 @@
     <axis xyz="0 0 1"/>
   </joint>
+  <joint name="front_laser_joint" type="fixed">
+        <parent link="base_link"/>
+        <child link="front_laser_link"/>
+        <origin xyz="-0.25 0.0 0.04" rpy="0 0 ${pi}"/>
+    </joint>
+    <link name="front_laser_link">
+        <visual>
+            <geometry>
+                <box size="0.01 0.01 0.01" />
+            </geometry>
+            <material name="red" />
+        </visual>
+    </link>
+  <xacro:include filename="lasers_def.xacro" />
+  <xacro:laser_sensor sensor_name="front" name="$(arg name)" />
   <!-- <joint name="caster_wheel_joint" type="continuous">
     <parent link="base_link"/>

Commit message: I have put KapiBara in sepearate namespace but it doesn't help a mouse is still stealing sensors

File: gazebo/src/workspace/src/gym/description/mouse.urdf.xacro (robot description, xacro)
@@ -84,5 +84,5 @@
     <parent link="base_link"/>
     <child link="left_wheel_link"/>
-    <origin xyz="-0.25 0.3 -0.15" rpy="${-pi/2} 0 0"/>
+    <origin xyz="-0.25 0.3 -0.15" rpy="${pi/2} 0 0"/>
     <axis xyz="0 0 1"/>
   </joint>
@@ -90,5 +90,5 @@
     <parent link="base_link"/>
     <child link="right_wheel_link"/>
-    <origin xyz="-0.25 -0.3 -0.15" rpy="${-pi/2} 0 0"/>
+    <origin xyz="-0.25 -0.3 -0.15" rpy="${pi/2} 0 0"/>
     <axis xyz="0 0 1"/>
   </joint>
@@ -134,5 +134,5 @@
     <plugin name="$(arg name)_gazebo_ros2_control" filename="libgazebo_ros2_control.so">
       <ros>
-        <namespace>/$(arg name)</namespace>
+        <namespace>$(arg name)</namespace>
         <remapping>/tf:=/$(arg name)/tf</remapping>
       </ros>

File: gazebo/src/workspace/src/kapibara/description/camera.xacro (robot description, xacro)
@@ -41,6 +41,6 @@
             <plugin name="camera_controller" filename="libgazebo_ros_camera.so">
                 <ros>
-                <namespace>KapiBara</namespace>
-                <remapping>~/out:=camera</remapping>
+                    <namespace>KapiBara</namespace>
+                    <remapping>~/out:=camera</remapping>
                 </ros>
                 <frame_name>camera_link_optical</frame_name>

File: gazebo/src/workspace/src/kapibara/description/imu.xacro (robot description, xacro)
@@ -56,5 +56,5 @@
         <plugin name="kapibara_imu" filename="libgazebo_ros_imu_sensor.so">
             <ros>
-                <namespace>Gazebo</namespace>
+                <namespace>KapiBara</namespace>
                 <remapping>~/out:=imu</remapping>
             </ros>

File: gazebo/src/workspace/src/kapibara/description/lasers_def.xacro (robot description, xacro)
@@ -38,5 +38,5 @@
             <plugin name="${sensor_name}_laserscan" filename="libgazebo_ros_ray_sensor.so">
                 <ros>
-                <namespace>Gazebo</namespace>
+                <namespace>KapiBara</namespace>
                 <remapping>~/out:=${sensor_name}</remapping>
                 </ros>

File: gazebo/src/workspace/src/kapibara/description/ros2_control.xacro (robot description, xacro)
@@ -104,7 +104,8 @@
         <plugin name="gazebo_ros2_control" filename="libgazebo_ros2_control.so">
             <ros>
-                <namespace>/</namespace>
+                <namespace>KapiBara</namespace>
+                <remapping>/tf:=/KapiBara/tf</remapping>
             </ros>
-            <robot_param_node>/robot_state_publisher</robot_param_node>
+            <robot_param_node>/KapiBara/robot_state_publisher</robot_param_node>
             <parameters>$(find kapibara)/config/my_controllers.yaml</parameters>
             <parameters>$(find kapibara)/config/my_controllers_sim.yaml</parameters>
