Commit message: Trigger work in maze simulation and now when I just use reset_world odom works

File: gazebo/src/workspace/src/gym/description/landmine.urdf.xacro (robot description, xacro)
@@ -4,5 +4,6 @@
   <xacro:arg name="height" default="1" />
   <xacro:arg name="depth" default="1" />
-  <link name="base_link">
+  <xacro:arg name="topic" default="trigger0" />
+  <link name="mine_link">
     <visual>
       <geometry>
@@ -15,5 +16,5 @@
     <collision name="front_bumper_collision">
       <geometry>
-        <box size="$(arg width) $(arg height) $(arg depth)"/>
+        <box size="$(arg width) $(arg height) 0.02"/>
       </geometry>
     </collision>
@@ -23,26 +24,21 @@
     </inertial>
   </link>
-  <gazebo reference="base_link">
+  <gazebo reference="mine_link">
     <material>Gazebo/Red</material>
-    <static>true</static>
+    <!-- <static>true</static> -->
     <sensor type="contact" name="contact_sensor">
       <always_on>true</always_on>
-      <update_rate>50</update_rate>
+      <update_rate>1</update_rate>
       <contact>
-        <collision>front_bumper_collision</collision>
+        <collision>mine_link_fixed_joint_lump__front_bumper_collision_collision</collision>
       </contact>
       <plugin name="bumper_plugin" filename="libgazebo_ros_bumper.so">
-        <ros>
-          <namespace>/landmine</namespace>
-          <remapping>bumper_states:=/contact_states</remapping>
-        </ros>
+          <alwaysOn>true</alwaysOn>
+          <!-- <remapping>bumper_states:=/contact_states</remapping> -->
+          <frameName>mine_link</frameName>
+          <ros>
+          <remapping>/bumper_states:=/$(arg topic)</remapping>
+          </ros>
       </plugin>
-      <plugin name="gazebo_ros_state" filename="libgazebo_ros_state.so">
-      <ros>
-        <namespace>/landmine</namespace>
-        <argument>model_states:=model_states_demo</argument>
-      </ros>
-      <update_rate>1.0</update_rate>
-    </plugin>
     </sensor>
   </gazebo>

Commit message: Trigger works as intendend!

File: gazebo/src/workspace/src/gym/description/landmine.urdf.xacro (robot description, xacro)
@@ -15,7 +15,15 @@
     </visual>
     <collision name="front_bumper_collision">
+      <origin xyz="0.0 0.0 ${-$(arg depth)/2}" />
       <geometry>
-        <box size="$(arg width) $(arg height) 0.02"/>
+        <box size="$(arg width) $(arg height) 0.2"/>
       </geometry>
+    <!-- <surface>
+        <contact>
+          <collide_bitmask>0x0000</collide_bitmask>
+          <collide_without_contact>true</collide_without_contact>
+          <collide_without_contact_bitmask>0x0000</collide_without_contact_bitmask>
+        </contact>
+    </surface> -->
     </collision>
     <inertial>
@@ -24,10 +32,13 @@
     </inertial>
   </link>
+  <gazebo>
+    <static>true</static>
+  </gazebo>
   <gazebo reference="mine_link">
     <material>Gazebo/Red</material>
-    <!-- <static>true</static> -->
+    <static>true</static>
     <sensor type="contact" name="contact_sensor">
       <always_on>true</always_on>
-      <update_rate>1</update_rate>
+      <update_rate>10</update_rate>
       <contact>
         <collision>mine_link_fixed_joint_lump__front_bumper_collision_collision</collision>

File: gazebo/src/workspace/src/kapibara/description/lasers_def.xacro (robot description, xacro)
@@ -34,4 +34,5 @@
                     <stddev>0.01</stddev>
             </noise>
+            <!-- <collision_bitmask>0x02</collision_bitmask> -->
             </ray>
             <plugin name="${sensor_name}_laserscan" filename="libgazebo_ros_ray_sensor.so">
@@ -40,5 +41,5 @@
                 <remapping>~/out:=${sensor_name}</remapping>
                 </ros>
-                <output_type>sensor_msgs/Range</output_type>
+                <output_type>sensor_msgs/LaserScan</output_type>
                 <radiation_type>infrared</radiation_type>
                 <frame_name>${sensor_name}_laser</frame_name>

Commit message: Fixed camera joint position, the camera overlaped with body of robot

File: gazebo/src/workspace/src/gym/description/landmine.urdf.xacro (robot description, xacro)
@@ -46,5 +46,4 @@
       <plugin name="bumper_plugin" filename="libgazebo_ros_bumper.so">
           <alwaysOn>true</alwaysOn>
-          <!-- <remapping>bumper_states:=/contact_states</remapping> -->
           <frameName>mine_link</frameName>
           <ros>

File: gazebo/src/workspace/src/kapibara/description/camera.xacro (robot description, xacro)
@@ -17,5 +17,5 @@
         <parent link="camera_link"/>
         <child link="camera_link_optical"/>
-        <origin xyz="0 0 0" rpy="${-pi/2} 0 ${-pi/2}"/>
+        <origin xyz="0.5 0 0" rpy="${-pi/2} 0 ${-pi/2}"/>
     </joint>
     <link name="camera_link_optical">

Commit message: I am able to detect collision and remove point upon contact with robot

File: gazebo/src/workspace/src/gym/description/landmine.urdf.xacro (robot description, xacro)
@@ -14,5 +14,5 @@
       </material>
     </visual>
-    <collision name="front_bumper_collision">
+    <collision name="front_bumper_collision_$(arg topic)">
       <origin xyz="0.0 0.0 ${-$(arg depth)/2}" />
       <geometry>
@@ -42,5 +42,5 @@
       <update_rate>10</update_rate>
       <contact>
-        <collision>mine_link_fixed_joint_lump__front_bumper_collision_collision</collision>
+        <collision>mine_link_fixed_joint_lump__front_bumper_collision_$(arg topic)_collision</collision>
       </contact>
       <plugin name="bumper_plugin_$(arg topic)" filename="libgazebo_ros_bumper.so">

Commit message: I am starting on doing parking simulation

File: gazebo/src/workspace/src/gym/description/landmine.urdf.xacro (robot description, xacro)
@@ -5,4 +5,5 @@
   <xacro:arg name="depth" default="1" />
   <xacro:arg name="topic" default="trigger0" />
+  <xacro:arg name="color" default="Red" />
   <link name="mine_link">
     <visual>
@@ -36,5 +37,5 @@
   </gazebo>
   <gazebo reference="mine_link">
-    <material>Gazebo/Red</material>
+    <material>Gazebo/$(arg color)</material>
     <static>true</static>
     <sensor type="contact" name="contact_sensor">

Commit message: I have added bumper sensor to mouse robot

File: gazebo/src/workspace/src/gym/description/landmine.urdf.xacro (robot description, xacro)
@@ -49,5 +49,5 @@
           <frameName>mine_link</frameName>
           <ros>
-          <remapping>/bumper_states:=/$(arg topic)</remapping>
+          <remapping>bumper_states:=$(arg topic)</remapping>
           </ros>
       </plugin>

File: gazebo/src/workspace/src/gym/description/mouse.urdf.xacro (robot description, xacro)
@@ -14,5 +14,5 @@
       <material name="blue"/>
     </visual>
-    <collision>
+    <collision name="base_link_collision_$(arg name)">
       <geometry>
         <box size="0.5 0.5 0.5"/>
@@ -21,5 +21,20 @@
   </link>
   <gazebo reference="base_link">
-        <material>Gazebo/Red</material>
+      <material>Gazebo/Red</material>
+      <sensor type="contact" name="contact_sensor">
+        <always_on>true</always_on>
+        <update_rate>10</update_rate>
+        <contact>
+          <collision>base_link_collision_$(arg name)_collision</collision>
+        </contact>
+        <plugin name="bumper_plugin_$(arg name)" filename="libgazebo_ros_bumper.so">
+            <alwaysOn>true</alwaysOn>
+            <frameName>base_link</frameName>
+            <ros>
+              <!-- <namespace>$(arg name)</namespace> -->
+              <remapping>bumper_states:=collision</remapping>
+            </ros>
+        </plugin>
+      </sensor>
   </gazebo>
   <link name="left_wheel_link">
