Commit message: I have fixed mouse URDF

File: gazebo/src/workspace/src/gym/description/lasers_def.xacro (robot description, xacro)
@@ -38,5 +38,5 @@
             <plugin name="${sensor_name}_laserscan" filename="libgazebo_ros_ray_sensor.so">
                 <ros>
-                <!-- <namespace>${name}</namespace> -->
+                <namespace>${name}</namespace>
                 <remapping>~/out:=${sensor_name}</remapping>
                 </ros>

File: gazebo/src/workspace/src/gym/description/mouse.urdf.xacro (robot description, xacro)
@@ -61,11 +61,11 @@
         <material>Gazebo/Black</material>
   </gazebo>
-  <!-- <link name="caster_wheel_link">
-    <xacro:inertial_sphere mass="0.1" radius="0.05">
+  <link name="caster_wheel_link">
+    <xacro:inertial_sphere mass="0.1" radius="0.1">
         <origin xyz="0 0 0" rpy="0 0 0" />
     </xacro:inertial_sphere>
     <visual>
       <geometry>
-        <sphere radius="0.05"/>
+        <sphere radius="0.1"/>
       </geometry>
       <material name="grey"/>
@@ -73,10 +73,12 @@
     <collision>
       <geometry>
-        <sphere radius="0.05"/>
+        <sphere radius="0.1"/>
       </geometry>
     </collision>
-  </link> -->
+  </link>
   <gazebo reference="caster_wheel_link">
         <material>Gazebo/Black</material>
+        <mu1 value="0.01"/>
+        <mu2 value="0.01"/>
   </gazebo>
   <!-- Joint Definitions -->
@@ -84,5 +86,5 @@
     <parent link="base_link"/>
     <child link="left_wheel_link"/>
-    <origin xyz="-0.25 0.3 -0.15" rpy="${pi/2} 0 0"/>
+    <origin xyz="-0.25 0.3 -0.19" rpy="${pi/2} 0 0"/>
     <axis xyz="0 0 1"/>
   </joint>
@@ -90,5 +92,5 @@
     <parent link="base_link"/>
     <child link="right_wheel_link"/>
-    <origin xyz="-0.25 -0.3 -0.15" rpy="${pi/2} 0 0"/>
+    <origin xyz="-0.25 -0.3 -0.19" rpy="${pi/2} 0 0"/>
     <axis xyz="0 0 1"/>
   </joint>
@@ -108,10 +110,10 @@
   <xacro:include filename="lasers_def.xacro" />
   <xacro:laser_sensor sensor_name="front" name="$(arg name)" />
-  <!-- <joint name="caster_wheel_joint" type="continuous">
+  <joint name="caster_wheel_joint" type="continuous">
     <parent link="base_link"/>
     <child link="caster_wheel_link"/>
-    <origin xyz="0 0 -0.05"/>
+    <origin xyz="0.22 0 -0.20"/>
     <axis xyz="0 0 1"/>
-  </joint> -->
+  </joint>
   <!-- ros2_control Configuration -->
   <ros2_control name="GazeboSystem_$(arg name)" type="system">
@@ -134,5 +136,5 @@
     <plugin name="$(arg name)_gazebo_ros2_control" filename="libgazebo_ros2_control.so">
       <ros>
-        <!-- <namespace>$(arg name)</namespace> -->
+        <namespace>$(arg name)</namespace>
         <remapping>/tf:=/$(arg name)/tf</remapping>
         <remapping>/tf_static:=/$(arg name)/tf_static</remapping>

File: gazebo/src/workspace/src/kapibara/description/camera.xacro (robot description, xacro)
@@ -41,5 +41,5 @@
             <plugin name="camera_controller" filename="libgazebo_ros_camera.so">
                 <ros>
-                    <!-- <namespace>KapiBara</namespace> -->
+                    <namespace>KapiBara</namespace>
                     <remapping>~/out:=camera</remapping>
                 </ros>

File: gazebo/src/workspace/src/kapibara/description/imu.xacro (robot description, xacro)
@@ -56,5 +56,5 @@
         <plugin name="kapibara_imu" filename="libgazebo_ros_imu_sensor.so">
             <ros>
-                <!-- <namespace>KapiBara</namespace> -->
+                <namespace>KapiBara</namespace>
                 <remapping>~/out:=imu</remapping>
             </ros>

File: gazebo/src/workspace/src/kapibara/description/lasers_def.xacro (robot description, xacro)
@@ -38,5 +38,5 @@
             <plugin name="${sensor_name}_laserscan" filename="libgazebo_ros_ray_sensor.so">
                 <ros>
-                    <!-- <namespace>KapiBara</namespace> -->
+                    <namespace>KapiBara</namespace>
                     <remapping>~/out:=${sensor_name}</remapping>
                 </ros>

File: gazebo/src/workspace/src/kapibara/description/ros2_control.xacro (robot description, xacro)
@@ -104,5 +104,5 @@
         <plugin name="kapibara_gazebo_ros2_control" filename="libgazebo_ros2_control.so">
             <ros>
-                <!-- <namespace>KapiBara</namespace> -->
+                <namespace>KapiBara</namespace>
                 <remapping>/tf:=/KapiBara/tf</remapping>
                 <remapping>/tf_static:=/KapiBara/tf_static</remapping>

Commit message: Mouse is moving in simulation

File: gazebo/src/workspace/src/gym/description/lasers_def.xacro (robot description, xacro)
@@ -14,6 +14,6 @@
                         <samples>20</samples>
                         <resolution>0.5</resolution>
-                        <min_angle>-0.22</min_angle>
-                        <max_angle>0.22</max_angle>
+                        <min_angle>-1</min_angle>
+                        <max_angle>1</max_angle>
                     </horizontal>
                     <vertical>

File: gazebo/src/workspace/src/gym/description/mouse.urdf.xacro (robot description, xacro)
@@ -12,5 +12,5 @@
         <box size="0.5 0.5 0.5"/>
       </geometry>
-      <material name="blue"/>
+      <material name="red"/>
     </visual>
     <collision name="base_link_collision_$(arg name)">
@@ -42,10 +42,10 @@
         <origin xyz="0 0 0" rpy="0 0 0" />
     </xacro:inertial_cylinder>
-    <visual>
+    <!-- <visual>
       <geometry>
         <cylinder length="0.1" radius="0.1"/>
       </geometry>
       <material name="black"/>
-    </visual>
+    </visual> -->
     <collision>
       <geometry>
@@ -61,10 +61,10 @@
         <origin xyz="0 0 0" rpy="0 0 0" />
     </xacro:inertial_cylinder>
-    <visual>
+    <!-- <visual>
       <geometry>
         <cylinder length="0.1" radius="0.1"/>
       </geometry>
       <material name="black"/>
-    </visual>
+    </visual> -->
     <collision>
       <geometry>
@@ -80,10 +80,10 @@
         <origin xyz="0 0 0" rpy="0 0 0" />
     </xacro:inertial_sphere>
-    <visual>
+    <!-- <visual>
       <geometry>
         <sphere radius="0.1"/>
       </geometry>
       <material name="grey"/>
-    </visual>
+    </visual> -->
     <collision>
       <geometry>
